File: Documentation/Hardware/Linear_Voltage_Regulator_6V/Linear_Voltage_Regulator.kicad_sch (KiCad schematic)
At the start: 12 parts, among them IC1 LDO, J1 Input 12V, J2 Output 6V, J3 Status LED, U1 Heatsink

Commit message: fixed schematic
Connections:
- net GND: now also J3.2; no longer J3.1
- net at R2.2: now also J3.1; no longer J3.2
Other:
- moved on the sheet: J3
Changed lines of the file:
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@@
 	(wire
 		(pts
-			(xy 191.77 119.38) (xy 191.77 127)
+			(xy 191.77 119.38) (xy 191.77 129.54)
 		)
 		(stroke
@@
 	(wire
 		(pts
-			(xy 194.31 124.46) (xy 196.85 124.46)
+			(xy 191.77 132.08) (xy 191.77 138.43)
 		)
 		(stroke
@@
 	(wire
 		(pts
-			(xy 194.31 121.92) (xy 194.31 124.46)
-		)
-		(stroke
-			(width 0)
-			(type default)
-		)
-	)
-	(wire
-		(pts
 			(xy 105.41 76.2) (xy 101.6 76.2)
 		)
@@
 		(pts
 			(xy 128.27 105.41) (xy 144.78 105.41)
-		)
-		(stroke
-			(width 0)
-			(type default)
-		)
-	)
-	(wire
-		(pts
-			(xy 191.77 127) (xy 196.85 127)
 		)
 		(stroke
@@
 	(symbol
 		(lib_id "power:GND")
-		(at 217.17 127 90)
+		(at 212.09 132.08 90)
 		(unit 1)
 		(exclude_from_sim no)
@@
 		(fields_autoplaced yes)
 		(property "Reference" "#PWR07"
-			(at 223.52 127 0)
+			(at 218.44 132.08 0)
 			(effects
 				(font
@@
 		)
 		(property "Value" "GND"
-			(at 220.98 126.9999 90)
+			(at 215.9 132.0799 90)
 			(effects
 				(font
@@
 		)
 		(property "Footprint" ""
-			(at 217.17 127 0)
+			(at 212.09 132.08 0)
 			(effects
 				(font
@@
 		)
 		(property "Datasheet" ""
-			(at 217.17 127 0)
+			(at 212.09 132.08 0)
 			(effects
 				(font
@@
 		)
 		(property "Description" "Power symbol creates a global label with name \"GND\" , ground"
-			(at 217.17 127 0)
+			(at 212.09 132.08 0)
 			(effects
 				(font
@@
 	(symbol
 		(lib_id "power:GND")
-		(at 194.31 121.92 180)
+		(at 191.77 138.43 0)
 		(unit 1)
 		(exclude_from_sim no)
@@
 		(fields_autoplaced yes)
 		(property "Reference" "#PWR05"
-			(at 194.31 115.57 0)
+			(at 191.77 144.78 0)
 			(effects
 				(font
@@
 		)
 		(property "Value" "GND"
-			(at 196.85 120.6499 0)
-			(effects
-				(font
-					(size 1.27 1.27)
-				)
-				(justify right)
+			(at 194.31 139.6999 0)
+			(effects
+				(font
+					(size 1.27 1.27)
+				)
+				(justify left)
 			)
 		)
 		(property "Footprint" ""
-			(at 194.31 121.92 0)
+			(at 191.77 138.43 0)
 			(effects
 				(font
@@
 		)
 		(property "Datasheet" ""
-			(at 194.31 121.92 0)
+			(at 191.77 138.43 0)
 			(effects
 				(font
@@
 		)
 		(property "Description" "Power symbol creates a global label with name \"GND\" , ground"
-			(at 194.31 121.92 0)
+			(at 191.77 138.43 0)
 			(effects
 				(font
@@
 	(symbol
 		(lib_id "power:GND")
-		(at 217.17 124.46 90)
+		(at 212.09 129.54 90)
 		(unit 1)
 		(exclude_from_sim no)
@@
 		(fields_autoplaced yes)
 		(property "Reference" "#PWR08"
-			(at 223.52 124.46 0)
+			(at 218.44 129.54 0)
 			(effects
 				(font
@@
 		)
 		(property "Value" "GND"
-			(at 220.98 124.4599 90)
+			(at 215.9 129.5399 90)
 			(effects
 				(font
@@
 		)
 		(property "Footprint" ""
-			(at 217.17 124.46 0)
+			(at 212.09 129.54 0)
 			(effects
 				(font
@@
 		)
 		(property "Datasheet" ""
-			(at 217.17 124.46 0)
+			(at 212.09 129.54 0)
 			(effects
 				(font
@@
 		)
 		(property "Description" "Power symbol creates a global label with name \"GND\" , ground"
-			(at 217.17 124.46 0)
+			(at 212.09 129.54 0)
 			(effects
 				(font
@@
 	(symbol
 		(lib_id "43650-0211:43650-0211")
-		(at 217.17 127 180)
+		(at 212.09 132.08 180)
 		(unit 1)
 		(exclude_from_sim no)
@@
 		(fields_autoplaced yes)
 		(property "Reference" "J3"
-			(at 207.01 116.84 0)
+			(at 201.93 121.92 0)
 			(effects
 				(font
@@
 		)
 		(property "Value" "Status LED"
-			(at 207.01 119.38 0)
+			(at 201.93 124.46 0)
 			(effects
 				(font
@@
 		)
 		(property "Footprint" "Molex_Microfit_2Pin:43650-02YY_091011"
-			(at 200.66 32.08 0)
+			(at 195.58 37.16 0)
 			(effects
 				(font
@@
 		)
 		(property "Datasheet" "https://www.molex.com/pdm_docs/sd/436500209_sd.pdf"
-			(at 200.66 -67.92 0)
+			(at 195.58 -62.84 0)
 			(effects
 				(font
@@
 		)
 		(property "Description" "Micro-Fit 3.0 Right-Angle Header, 3.00mm Pitch, Single Row, 2 Circuits, with PCB Press-fit Metal Retention Clip, Glow-Wire Capable, Black, Tape and Reel"
-			(at 217.17 127 0)
+			(at 212.09 132.08 0)
 			(effects
 				(font
@@
 		)
 		(property "Height" "5.57"
-			(at 200.66 -267.92 0)
+			(at 195.58 -262.84 0)
 			(effects
 				(font
@@
 		)
 		(property "Mouser Part Number" "538-43650-0211"
-			(at 200.66 -367.92 0)
+			(at 195.58 -362.84 0)
 			(effects
 				(font
@@
 		)
 		(property "Mouser Price/Stock" "https://www.mouser.co.uk/ProductDetail/Molex/43650-0211?qs=z57USrEQgt0F0sS1hGS9Bw%3D%3D"
-			(at 200.66 -467.92 0)
+			(at 195.58 -462.84 0)
 			(effects
 				(font
@@
 		)
 		(property "Manufacturer_Name" "Molex"
-			(at 200.66 -567.92 0)
+			(at 195.58 -562.84 0)
 			(effects
 				(font
@@
 		)
 		(property "Manufacturer_Part_Number" "43650-0211"
-			(at 200.66 -667.92 0)
-			(effects
-				(font
+			(at 195.58 -662.84 0)
+			(effects
+				(font
